File: esp-card.kicad_pcb (KiCad board)
At the start: 2 copper layers, 0 parts

Commit message: symbol fixes + placement
Parts:
- added AE1: Antenna, ESP_Antenna:ESPRESSIF_ESP32_MIFA_2.4GHz_Right, F.Cu at (200.6, 104.7)
- added C1: 1uF, Capacitor_SMD:C_0402_1005Metric, F.Cu at (132.1, 96.5)
- added C10: 100nF, Capacitor_SMD:C_0402_1005Metric, F.Cu at (159.2, 64.1)
- added C11: 100nF, Capacitor_SMD:C_0402_1005Metric, F.Cu at (159.2, 66.0)
- added C12: 2.2uF, Capacitor_SMD:C_0402_1005Metric, F.Cu at (159.2, 68.0)
- added C13: 100nF, Capacitor_SMD:C_0402_1005Metric, F.Cu at (161.9, 61.5)
- added C14: 100nF, Capacitor_SMD:C_0402_1005Metric, F.Cu at (162.1, 64.1)
- added C15: 1uF, Capacitor_SMD:C_0402_1005Metric, F.Cu at (162.1, 66.0)
- added C16: 2.2uF, Capacitor_SMD:C_0402_1005Metric, F.Cu at (162.1, 68.0)
- added C2: 1uF, Capacitor_SMD:C_0402_1005Metric, F.Cu at (119.4, 99.1)
- added C3: 12pF, Capacitor_SMD:C_0402_1005Metric, F.Cu at (153.5, 66.0)
- added C4: 12pF, Capacitor_SMD:C_0402_1005Metric, F.Cu at (153.5, 68.0)
- added C5: 10pF, Capacitor_SMD:C_0402_1005Metric, F.Cu at (156.3, 62.1)
- added C6: 100nF, Capacitor_SMD:C_0402_1005Metric, F.Cu at (134.6, 98.6)
- added C7: 2pF, Capacitor_SMD:C_0402_1005Metric, F.Cu at (187.5, 96.5)
- added C8: 2pF, Capacitor_SMD:C_0402_1005Metric, F.Cu at (156.3, 68.0)
- added C9: 1uF, Capacitor_SMD:C_0402_1005Metric, F.Cu at (159.2, 62.1)
- added J2: Conn_01x04_Socket, Connector_PinHeader_2.54mm:PinHeader_1x04_P2.54mm_Vertical, F.Cu at (134.6, 71.1)
- added L1: 2nH, Inductor_SMD:L_0402_1005Metric, F.Cu at (182.4, 101.6)
- added L2: 2nH, Inductor_SMD:L_0402_1005Metric, F.Cu at (138.4, 116.8)
- added R1: 5.1k, Resistor_SMD:R_0402_1005Metric, F.Cu at (126.5, 78.7)
- added R2: 5.1k, Resistor_SMD:R_0402_1005Metric, F.Cu at (146.8, 109.2)
- added R3: 1.5k, Resistor_SMD:R_0402_1005Metric, F.Cu at (129.0, 86.4)
- added R4: 10k, Resistor_SMD:R_0402_1005Metric, F.Cu at (149.9, 102.1)
- added R5: 10k, Resistor_SMD:R_0402_1005Metric, F.Cu at (146.8, 104.1)
- added R6: 0, Resistor_SMD:R_0402_1005Metric, F.Cu at (192.5, 106.7)
- added R7: 0, Resistor_SMD:R_0402_1005Metric, F.Cu at (195.1, 109.2)
- added U1: NH-B1010RGBT-HF, footprint:LED-ARRAY-SMD_4P-L1.0-W1.0-TR_NH-B1010RGBT, F.Cu at (191.5, 65.2)
- added U2: ESP32-C3FH4, footprint:QFN-32_L5.0-W5.0-P0.50-TL-EP3.7, F.Cu at (139.7, 88.9)
- added U3: NH-B1010RGBT-HF, footprint:LED-ARRAY-SMD_4P-L1.0-W1.0-TR_NH-B1010RGBT, F.Cu at (191.5, 68.1)
- added U4: TS-1187A-B-A-B, footprint:SW-SMD_4P-L5.1-W5.1-P3.70-LS6.5-TL-2, F.Cu at (160.0, 99.1)
- added U58: TS-1187A-B-A-B, footprint:SW-SMD_4P-L5.1-W5.1-P3.70-LS6.5-TL-2, F.Cu at (139.7, 99.1)
- added U59: YTC-TC16-30, footprint:USB-C-SMD_YIYUAN_YTC-TC16-30, F.Cu at (121.9, 86.4)
- added U60: AMS1117-3_3, footprint:SOT-223-3_L6.5-W3.4-P2.30-LS7.0-BR, F.Cu at (124.5, 101.6)
- added U61: NH-B1010RGBT-HF, footprint:LED-ARRAY-SMD_4P-L1.0-W1.0-TR_NH-B1010RGBT, F.Cu at (191.5, 71.1)
- added U62: NH-B1010RGBT-HF, footprint:LED-ARRAY-SMD_4P-L1.0-W1.0-TR_NH-B1010RGBT, F.Cu at (191.5, 74.0)
- added U63: NH-B1010RGBT-HF, footprint:LED-ARRAY-SMD_4P-L1.0-W1.0-TR_NH-B1010RGBT, F.Cu at (191.5, 77.0)
- added U64: NH-B1010RGBT-HF, footprint:LED-ARRAY-SMD_4P-L1.0-W1.0-TR_NH-B1010RGBT, F.Cu at (195.2, 65.2)
- added U65: NH-B1010RGBT-HF, footprint:LED-ARRAY-SMD_4P-L1.0-W1.0-TR_NH-B1010RGBT, F.Cu at (195.2, 68.1)
- added U66: NH-B1010RGBT-HF, footprint:LED-ARRAY-SMD_4P-L1.0-W1.0-TR_NH-B1010RGBT, F.Cu at (195.2, 71.1)
- added U67: NH-B1010RGBT-HF, footprint:LED-ARRAY-SMD_4P-L1.0-W1.0-TR_NH-B1010RGBT, F.Cu at (195.2, 74.0)
- added U68: NH-B1010RGBT-HF, footprint:LED-ARRAY-SMD_4P-L1.0-W1.0-TR_NH-B1010RGBT, F.Cu at (195.2, 77.0)
- added U69: NH-B1010RGBT-HF, footprint:LED-ARRAY-SMD_4P-L1.0-W1.0-TR_NH-B1010RGBT, F.Cu at (198.8, 65.2)
- added U70: NH-B1010RGBT-HF, footprint:LED-ARRAY-SMD_4P-L1.0-W1.0-TR_NH-B1010RGBT, F.Cu at (198.8, 68.1)
- added U71: NH-B1010RGBT-HF, footprint:LED-ARRAY-SMD_4P-L1.0-W1.0-TR_NH-B1010RGBT, F.Cu at (198.8, 71.1)
- added U72: NH-B1010RGBT-HF, footprint:LED-ARRAY-SMD_4P-L1.0-W1.0-TR_NH-B1010RGBT, F.Cu at (198.8, 74.0)
- added X1: CF4040M00015001, footprint:CRYSTAL-SMD_4P-L3.2-W2.5-BL_SIT8008BI, F.Cu at (144.8, 78.7)
Other:
- board outline added: 6.5 x 10.9 mm
