File: esp-card.kicad_pcb (KiCad board)
At the start: 2 copper layers, 6.5 x 10.9 mm, 47 parts, among them J2 Conn_01x04_Socket, U1 NH-B1010RGBT-HF, U2 ESP32-C3FH4, U3 NH-B1010RGBT-HF, U4 TS-1187A-B-A-B, U58 TS-1187A-B-A-B, U59 YTC-TC16-30, U60 AMS1117-3_3, U61 NH-B1010RGBT-HF, U62 NH-B1010RGBT-HF, U63 NH-B1010RGBT-HF, U64 NH-B1010RGBT-HF, U65 NH-B1010RGBT-HF, U66 NH-B1010RGBT-HF, U67 NH-B1010RGBT-HF, U68 NH-B1010RGBT-HF, U69 NH-B1010RGBT-HF, U70 NH-B1010RGBT-HF, U71 NH-B1010RGBT-HF, U72 NH-B1010RGBT-HF, X1 CF4040M00015001

Commit message: updated sheet
Parts:
- added C17: 100nF, Capacitor_SMD:C_0402_1005Metric, F.Cu at (150.6, 88.9)
- added C18: 100nF, Capacitor_SMD:C_0402_1005Metric, F.Cu at (165.1, 88.9)
- added R8: 10k, Resistor_SMD:R_0402_1005Metric, F.Cu at (161.3, 88.9)
- added R9: 10k, Resistor_SMD:R_0402_1005Metric, F.Cu at (180.3, 81.8)
- added U5: TS-1187A-B-A-B, footprint:SW-SMD_4P-L5.1-W5.1-P3.70-LS6.5-TL-2, F.Cu at (154.9, 88.9)
- added U73: TS-1187A-B-A-B, footprint:SW-SMD_4P-L5.1-W5.1-P3.70-LS6.5-TL-2, F.Cu at (172.0, 89.6)
- moved L2 26.5 mm to (121.4, 96.5)
- moved C1 3.59 mm to (129.5, 99.1)
- moved U60 2.54 mm to (124.5, 99.1)
Connections:
- net /CTRL0 renamed /LED_Matrix_7_pin/CTRL0
- net /CTRL1 renamed /LED_Matrix_7_pin/CTRL1
- net /CTRL2 renamed /LED_Matrix_7_pin/CTRL2
- net /CTRL3 renamed /LED_Matrix_7_pin/CTRL3
- net /CTRL4 renamed /LED_Matrix_7_pin/CTRL4
- net /CTRL5 renamed /LED_Matrix_7_pin/CTRL5
- net /CTRL6 renamed /LED_Matrix_7_pin/CTRL6
- net G10 renamed /ESP32/G10
- AE1 pad 2: (no net) -> GND
- U2 pad 14: /ESP32/G8 -> GPIO8
- U2 pad 6: G2 -> GPIO2

Commit message: fixed LED matrix
Parts:
- added L3: 3.9nH, Inductor_SMD:L_0402_1005Metric, F.Cu at (121.4, 95.5)
- L2: value 2nH -> 3.9nH
- moved C8 39.2 mm to (181.9, 97.8)
- moved C5 37.0 mm to (154.9, 99.1), turned to -90 degrees
- moved C16 36.9 mm to (133.3, 91.2), turned to 180 degrees
- moved C10 36.1 mm to (137.2, 92.7), turned to 180 degrees
- moved U64 36.1 mm to (230.4, 57.2)
- moved U65 36.1 mm to (230.4, 60.2)
- moved U66 36.1 mm to (230.4, 63.1)
- moved U67 36.1 mm to (230.4, 66.1)
- moved U68 36.1 mm to (230.4, 69.0)
- moved U69 36.1 mm to (234.1, 57.2)
- moved U70 36.1 mm to (234.1, 60.2)
- moved U71 36.1 mm to (234.1, 63.1)
- moved U72 36.1 mm to (234.1, 66.1)
- moved U1 36.1 mm to (226.8, 57.2)
- moved U3 36.1 mm to (226.8, 60.2)
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Connections:
- C10 pad 1: Net-(C10-Pad1) -> Net-(D2-A)
- L2 pad 2: Net-(C10-Pad1) -> Net-(D2-A)
- U2 pad 10: G5 -> /LED_Matrix_7_pin/CTRL4
- U2 pad 12: G6 -> /LED_Matrix_7_pin/CTRL5
- U2 pad 13: /ESP32/G7 -> /LED_Matrix_7_pin/CTRL6
- U2 pad 2: Net-(C10-Pad1) -> Net-(D2-K)
- U2 pad 3: Net-(C10-Pad1) -> Net-(D2-K)
- U2 pad 31: +3.3V -> Net-(D1-K)
- U2 pad 32: +3.3V -> Net-(D1-K)
- U2 pad 4: G0 -> /LED_Matrix_7_pin/CTRL0
- U2 pad 5: G1 -> /LED_Matrix_7_pin/CTRL1
- U2 pad 8: G3 -> /LED_Matrix_7_pin/CTRL2
- U2 pad 9: G4 -> /LED_Matrix_7_pin/CTRL3
Other:
- board size 6.5 x 10.9 mm -> 85 x 55 mm

Commit message: fixed LED matrix
Parts:
- moved C14 41.3 mm to (133.3, 93.7), turned to 180 degrees
- moved C13 39.4 mm to (133.3, 88.6), turned to 180 degrees
- moved C15 37.2 mm to (133.4, 89.7), turned to 180 degrees
- moved C10 4.47 mm to (133.3, 95.0)
- moved C11 1.52 mm to (133.3, 90.7)
- moved C12 1.52 mm to (133.3, 91.7)
- moved C16 1.52 mm to (133.3, 92.7)
Connections:
- U2 pad 31: Net-(D1-K) -> +3.3V
- U2 pad 32: Net-(D1-K) -> +3.3V

Commit message: better routing
Parts:
- L1: value 2nH -> 2.2nH
- moved U1 76.8 mm to (166.9, 105.4)
- moved U3 76.8 mm to (166.9, 108.3)
- moved U64 76.8 mm to (170.6, 105.4)
- moved U65 76.8 mm to (170.6, 108.3)
- moved U69 76.8 mm to (174.2, 105.4)
- moved U70 76.8 mm to (174.2, 108.3)
- moved U61 76.8 mm to (166.9, 111.3)
- moved U62 76.8 mm to (166.9, 114.2)
- moved U63 76.8 mm to (166.9, 117.2)
- moved U66 76.8 mm to (170.6, 111.3)
- moved U67 76.8 mm to (170.6, 114.2)
- moved U68 76.8 mm to (170.6, 117.2)
- moved U71 76.8 mm to (174.2, 111.3)
- moved U72 76.8 mm to (174.2, 114.2)
- moved R9 47.4 mm to (148.1, 116.5), turned to -90 degrees
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Connections:
- C10 pad 1: Net-(D2-A) -> Net-(C10-Pad1)
- L2 pad 2: Net-(D2-A) -> Net-(C10-Pad1)
- L3 pad 2: Net-(D2-A) -> Net-(C10-Pad1)
- U2 pad 2: Net-(D2-K) -> Net-(C10-Pad1)
- U2 pad 3: Net-(D2-K) -> Net-(C10-Pad1)
Routing:
- net GND: track 0.00 -> 3.05 mm

Commit message: fixed routing
Parts:
- moved C6 25.4 mm to (149.1, 117.3), turned to 90 degrees
- moved C17 24.1 mm to (148.1, 125.0), turned to 90 degrees
- moved R4 22.6 mm to (127.3, 117.0), turned to 90 degrees
- moved R9 22.5 mm to (127.3, 125.0), turned to 90 degrees
- moved U58 16.5 mm to (144.0, 116.8), turned to 180 degrees
- moved U5 16.4 mm to (143.8, 125.0), turned to 180 degrees
- moved U4 14.3 mm to (132.1, 117.0), turned to 180 degrees
- moved U73 14.1 mm to (132.1, 125.0), turned to 180 degrees
- moved R5 9.78 mm to (139.2, 116.8), turned to 90 degrees
- moved R8 9.48 mm to (138.9, 124.7), turned to 90 degrees
- moved C5 9.07 mm to (136.9, 117.0), turned to 90 degrees
- moved C18 9.07 mm to (136.9, 125.2), turned to 90 degrees
- moved C9 8.73 mm to (144.3, 101.3), turned to 0 degrees
- moved J2 8.64 mm to (136.1, 76.2), turned to -90 degrees
- moved C1 8.49 mm to (112.3, 108.9)
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Routing:
- net +5V: track 0.00 -> 81.0 mm, vias 0 -> 3
- net ANT: track 0.00 -> 59.4 mm, vias 0 -> 2
- net GND: track 3.05 -> 52.9 mm, vias 0 -> 1
- net UART_0_TX: track 0.00 -> 31.3 mm, vias 0 -> 1
- net UART_0_RX: track 0.00 -> 31.2 mm, vias 0 -> 1
- net USB_N: track 0.00 -> 24.9 mm
- net +3.3V: track 0.00 -> 17.7 mm
- net USB_PU: track 0.00 -> 14.0 mm
- net Net-(C10-Pad1): track 0.00 -> 12.3 mm, vias 0 -> 2
- net Net-(U59-DP1): track 0.00 -> 10.7 mm, vias 0 -> 3
- net XOUT: track 0.00 -> 9.64 mm, vias 0 -> 2
- net XIN: track 0.00 -> 8.10 mm
- net Net-(U59-CC1): track 0.00 -> 3.27 mm
- net Net-(U58-C): track 0.00 -> 2.59 mm
- net Net-(U59-CC2): track 0.00 -> 2.46 mm
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
Commit message: antenna footprint fix
Parts:
- moved U3 38.4 mm to (138.8, 82.2), turned to -90 degrees
- moved C6 36.9 mm to (112.8, 123.9), turned to -90 degrees
- moved C17 35.4 mm to (113.8, 116.2), turned to -90 degrees
- moved U1 33.1 mm to (133.8, 107.2), turned to 135 degrees
- moved U58 27.2 mm to (117.9, 124.4), turned to 0 degrees
- moved U5 27.1 mm to (118.1, 116.2), turned to 0 degrees
- moved R5 18.1 mm to (122.7, 124.3), turned to -90 degrees
- moved R8 18.0 mm to (122.9, 116.5), turned to -90 degrees
- moved C18 15.1 mm to (125.0, 116.0), turned to -90 degrees
- moved C5 14.0 mm to (125.0, 124.2), turned to -90 degrees
- moved U62 13.0 mm to (164.5, 101.5)
- moved U61 12.9 mm to (167.8, 98.4), turned to 180 degrees
- moved U63 12.4 mm to (159.1, 107.6)
- moved R9 11.4 mm to (134.6, 116.2), turned to -90 degrees
- moved R4 10.3 mm to (134.6, 124.2), turned to -90 degrees
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Connections:
- R1 pad 1: GND -> Net-(U59-CC1)
- R1 pad 2: Net-(U59-CC1) -> GND
Routing:
- net /LED_Matrix_7_pin/CTRL0: track 0.00 -> 29.8 mm, vias 0 -> 2
- net /LED_Matrix_7_pin/CTRL3: track 0.00 -> 26.6 mm, vias 0 -> 3
- net /LED_Matrix_7_pin/CTRL1: track 0.00 -> 25.9 mm, vias 0 -> 2
- net EN: track 2.08 -> 26.4 mm, vias 0 -> 2
- net /LED_Matrix_7_pin/CTRL2: track 0.00 -> 24.0 mm, vias 0 -> 2
- net GPIO9: track 2.08 -> 25.3 mm
- net /LED_Matrix_7_pin/CTRL4: track 0.00 -> 20.8 mm, vias 0 -> 2
- net +3.3V: track 17.7 -> 38.4 mm
- net GND: track 52.9 -> 33.5 mm, vias 1 -> 7
- net GPIO2: track 2.23 -> 21.1 mm, vias 0 -> 2
- net /LED_Matrix_7_pin/CTRL5: track 0.00 -> 18.6 mm, vias 0 -> 2
- net /LED_Matrix_7_pin/CTRL6: track 0.00 -> 17.3 mm, vias 0 -> 2
- net GPIO8: track 0.00 -> 16.8 mm
- net +5V: track 81.0 -> 67.8 mm, vias 3 -> 5
- net Net-(C10-Pad1): track 12.3 -> 4.86 mm, vias 2 -> 0
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- added copper zone on B.Cu, net GND

Commit message: finished up routing
Parts:
- moved U408 29.4 mm to (163.5, 98.2)
- moved U402 20.3 mm to (167.5, 78.1), turned to 0 degrees
- moved J1 19.4 mm to (130.3, 94.7), turned to 90 degrees
- moved U412 17.8 mm to (160.5, 98.2), turned to -90 degrees
- moved U407 15.6 mm to (163.5, 95.2), turned to -90 degrees
- moved U411 15.3 mm to (160.5, 95.2), turned to -90 degrees
- moved U403 14.4 mm to (166.5, 95.2), turned to -90 degrees
- moved U414 13.8 mm to (160.5, 104.2), turned to -90 degrees
- moved U413 12.7 mm to (160.5, 101.2), turned to -90 degrees
- moved U405 9.96 mm to (166.5, 101.2), turned to -90 degrees
- moved U404 7.18 mm to (166.5, 98.2), turned to -90 degrees
- moved U406 6.52 mm to (166.5, 104.2), turned to -90 degrees
- moved U410 5.91 mm to (163.5, 104.2), turned to -90 degrees
- moved U409 1.05 mm to (163.5, 101.2), turned to -90 degrees
- renumbered C17 to C10, C18 to C11, C9 to C12, C14 to C13, C5 to C14, C6 to C15, C13 to C16, C15 to C17, C16 to C18, C3 to C2, C2 to C3, C12 to C5, C11 to C6, C10 to C7, C7 to C8, C8 to C9, J2 to J1, L3 to L1, L1 to L3, R6 to R4, R7 to R5, R8 to R6, R9 to R7, R4 to R8, R5 to R9, U1 to U401, U61 to U402, U63 to U403, U65 to U404, U67 to U405, U69 to U406, U71 to U407, U3 to U408, U62 to U409, U64 to U410, U66 to U411, U68 to U412, U70 to U413, U72 to U414, U60 to U53, U59 to U54, U2 to U55, U5 to U56, U73 to U57, U4 to U58, U58 to U59
Routing:
- net /LED_Matrix_7_pin/CTRL1: track 25.9 -> 116.2 mm, vias 2 -> 10
- net /LED_Matrix_7_pin/CTRL3: track 26.6 -> 112.6 mm, vias 3 -> 8
- net /LED_Matrix_7_pin/CTRL2: track 24.0 -> 100.6 mm, vias 2 -> 8
- net /LED_Matrix_7_pin/CTRL0: track 29.8 -> 87.6 mm, vias 2 -> 5
- net /LED_Matrix_7_pin/CTRL6: track 17.3 -> 61.6 mm, vias 2 -> 7
- net /LED_Matrix_7_pin/CTRL4: track 20.8 -> 57.2 mm, vias 2 -> 9
- net /LED_Matrix_7_pin/CTRL5: track 18.6 -> 52.6 mm, vias 2 -> 12
- net UART_0_RX: track 31.2 -> 6.06 mm
- net UART_0_TX: track 31.3 -> 6.62 mm
- net GND: track 33.5 -> 9.50 mm, vias 7 -> 1
- net +3.3V: track 38.4 -> 29.0 mm, vias 0 -> 2
- net ANT: track 58.2 -> 59.3 mm
- added copper zone on F.Cu, net +3.3V
- added copper zone on F.Cu, net GND
Other:
- board text added: "Embedded/Full-Stack Developer"
- board text added: "VIncent Xie"

Commit message: DRC checks
Parts:
- moved C4 0.51 mm to (127.0, 98.7)
- moved R3 0.45 mm to (122.8, 99.6), turned to 45 degrees
- moved U53 0.12 mm to (122.1, 109.5)
- moved U54 0.12 mm to (114.8, 101.6)
Routing:
- net ANT: track 59.3 -> 67.4 mm
- net Net-(AE1-A): track 0.22 -> 6.72 mm
- net GND: track 9.50 -> 14.1 mm
- net XOUT: track 11.4 -> 15.6 mm
- net /LED_Matrix_7_pin/CTRL5: track 52.6 -> 56.0 mm
- net Net-(R4-Pad2): track 0.00 -> 1.27 mm
- net USB_PU: track 14.0 -> 14.7 mm
- net /LED_Matrix_7_pin/CTRL2: track 100.6 -> 101.2 mm
- net /LED_Matrix_7_pin/CTRL0: track 87.6 -> 87.1 mm
Other:
- outline, holes or cut-outs redrawn
