File: esp-card.kicad_sch (KiCad schematic)
At the start: 0 parts

Commit message: fixed LED matrix
Connections:
- no-connect marks 3 -> 2
Other:
- sheet ESP32 ports: added G10; removed G7, G8
- sheet LED_Matrix_7_pin ports: added input0, input1, input2, input3, input4, input5, input6; removed Input[0..6]
