File: ESP32.kicad_sch (KiCad schematic)
At the start: 40 parts, among them J2 Conn_01x04_Socket, U2 ESP32-C3FH4, U4 TS-1187A-B-A-B, U5 TS-1187A-B-A-B, U58 TS-1187A-B-A-B, U59 YTC-TC16-30, U60 AMS1117-3_3, U73 TS-1187A-B-A-B, X1 CF4040M00015001

Commit message: fixed routing
Connections:
- net GND: now also R1.2; no longer R1.1
- net at U59.A5 (CC1): now also R1.1; no longer R1.2
Other:
- moved on the sheet: R1
Changed lines of the file:
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@@
 	(symbol
 		(lib_id "Device:R")
-		(at 27.94 52.07 90)
+		(at 27.94 52.07 270)
+		(mirror x)
 		(unit 1)
 		(exclude_from_sim no)

Commit message: finished up routing
Parts:
- renumbered C17 to C10, C18 to C11, C9 to C12, C14 to C13, C5 to C14, C6 to C15, C13 to C16, C15 to C17, C16 to C18, C3 to C2, C2 to C3, C12 to C5, C11 to C6, C10 to C7, C7 to C8, C8 to C9, J2 to J1, L3 to L1, L1 to L3, R6 to R4, R7 to R5, R8 to R6, R9 to R7, R4 to R8, R5 to R9, U60 to U53, U59 to U54, U2 to U55, U5 to U56, U73 to U57, U4 to U58, U58 to U59
