File: LED_Matrix_7_pin.kicad_sch (KiCad schematic)
At the start: 14 parts, among them U1 NH-B1010RGBT-HF, U3 NH-B1010RGBT-HF, U61 NH-B1010RGBT-HF, U62 NH-B1010RGBT-HF, U63 NH-B1010RGBT-HF, U64 NH-B1010RGBT-HF, U65 NH-B1010RGBT-HF, U66 NH-B1010RGBT-HF, U67 NH-B1010RGBT-HF, U68 NH-B1010RGBT-HF, U69 NH-B1010RGBT-HF, U70 NH-B1010RGBT-HF, U71 NH-B1010RGBT-HF, U72 NH-B1010RGBT-HF

Commit message: fixed LED matrix
Connections:
- net CTRL0 renamed input0
- net CTRL1 renamed input1
- net CTRL2 renamed input2
- net CTRL3 renamed input3
- net CTRL4 renamed input4
- net CTRL5 renamed input5
- net CTRL6 renamed input6

Commit message: finished up routing
Parts:
- renumbered U1 to U401, U61 to U402, U63 to U403, U65 to U404, U67 to U405, U69 to U406, U71 to U407, U3 to U408, U62 to U409, U64 to U410, U66 to U411, U68 to U412, U70 to U413, U72 to U414
Changed lines of the file:
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@@
 		(dnp no)
 		(fields_autoplaced yes)
-		(property "Reference" "U70"
+		(property "Reference" "U413"
 			(at 88.9 196.85 0)
 			(effects
@@
 			(project "esp-card"
 				(path "/93cf1a11-1660-4ae3-a523-02ca090cff0a/8f237209-f932-45f7-b7bc-f97443ee2306"
-					(reference "U70")
+					(reference "U413")
 					(unit 1)
 				)
@@
 		(dnp no)
 		(fields_autoplaced yes)
-		(property "Reference" "U1"
+		(property "Reference" "U401"
 			(at 52.07 38.1 0)
 			(effects
@@
 			(project "esp-card"
 				(path "/93cf1a11-1660-4ae3-a523-02ca090cff0a/8f237209-f932-45f7-b7bc-f97443ee2306"
-					(reference "U1")
+					(reference "U401")
 					(unit 1)
 				)
@@
 		(dnp no)
 		(fields_autoplaced yes)
-		(property "Reference" "U66"
+		(property "Reference" "U411"
 			(at 88.9 133.35 0)
 			(effects
@@
 			(project "esp-card"
 				(path "/93cf1a11-1660-4ae3-a523-02ca090cff0a/8f237209-f932-45f7-b7bc-f97443ee2306"
-					(reference "U66")
+					(reference "U411")
 					(unit 1)
 				)
@@
 		(dnp no)
 		(fields_autoplaced yes)
-		(property "Reference" "U62"
+		(property "Reference" "U409"
 			(at 88.9 69.85 0)
 			(effects
@@
 			(project "esp-card"
 				(path "/93cf1a11-1660-4ae3-a523-02ca090cff0a/8f237209-f932-45f7-b7bc-f97443ee2306"
-					(reference "U62")
+					(reference "U409")
 					(unit 1)
 				)
@@
 		(dnp no)
 		(fields_autoplaced yes)
-		(property "Reference" "U72"
+		(property "Reference" "U414"
 			(at 88.9 228.6 0)
 			(effects
@@
 			(project "esp-card"
 				(path "/93cf1a11-1660-4ae3-a523-02ca090cff0a/8f237209-f932-45f7-b7bc-f97443ee2306"
-					(reference "U72")
+					(reference "U414")
 					(unit 1)
 				)
@@
 		(dnp no)
 		(fields_autoplaced yes)
-		(property "Reference" "U71"
+		(property "Reference" "U407"
 			(at 52.07 228.6 0)
 			(effects
@@
 			(project "esp-card"
 				(path "/93cf1a11-1660-4ae3-a523-02ca090cff0a/8f237209-f932-45f7-b7bc-f97443ee2306"
-					(reference "U71")
+					(reference "U407")
 					(unit 1)
 				)
@@
 		(dnp no)
 		(fields_autoplaced yes)
-		(property "Reference" "U3"
+		(property "Reference" "U408"
 			(at 88.9 38.1 0)
 			(effects
@@
 			(project "esp-card"
 				(path "/93cf1a11-1660-4ae3-a523-02ca090cff0a/8f237209-f932-45f7-b7bc-f97443ee2306"
-					(reference "U3")
+					(reference "U408")
 					(unit 1)
 				)
@@
 		(dnp no)
 		(fields_autoplaced yes)
-		(property "Reference" "U65"
+		(property "Reference" "U404"
 			(at 52.07 133.35 0)
 			(effects
@@
 			(project "esp-card"
 				(path "/93cf1a11-1660-4ae3-a523-02ca090cff0a/8f237209-f932-45f7-b7bc-f97443ee2306"
-					(reference "U65")
+					(reference "U404")
 					(unit 1)
 				)
@@
 		(dnp no)
 		(fields_autoplaced yes)
-		(property "Reference" "U68"
+		(property "Reference" "U412"
 			(at 88.9 165.1 0)
 			(effects
@@
 			(project "esp-card"
 				(path "/93cf1a11-1660-4ae3-a523-02ca090cff0a/8f237209-f932-45f7-b7bc-f97443ee2306"
-					(reference "U68")
+					(reference "U412")
 					(unit 1)
 				)
@@
 		(dnp no)
 		(fields_autoplaced yes)
-		(property "Reference" "U69"
+		(property "Reference" "U406"
 			(at 52.07 196.85 0)
 			(effects
@@
 			(project "esp-card"
 				(path "/93cf1a11-1660-4ae3-a523-02ca090cff0a/8f237209-f932-45f7-b7bc-f97443ee2306"
-					(reference "U69")
+					(reference "U406")
 					(unit 1)
 				)
@@
 		(dnp no)
 		(fields_autoplaced yes)
-		(property "Reference" "U64"
+		(property "Reference" "U410"
 			(at 88.9 101.6 0)
 			(effects
@@
 			(project "esp-card"
 				(path "/93cf1a11-1660-4ae3-a523-02ca090cff0a/8f237209-f932-45f7-b7bc-f97443ee2306"
-					(reference "U64")
+					(reference "U410")
 					(unit 1)
 				)
@@
 		(dnp no)
 		(fields_autoplaced yes)
-		(property "Reference" "U63"
+		(property "Reference" "U403"
 			(at 52.07 101.6 0)
 			(effects
@@
 			(project "esp-card"
 				(path "/93cf1a11-1660-4ae3-a523-02ca090cff0a/8f237209-f932-45f7-b7bc-f97443ee2306"
-					(reference "U63")
+					(reference "U403")
 					(unit 1)
 				)
@@
 		(dnp no)
 		(fields_autoplaced yes)
-		(property "Reference" "U67"
+		(property "Reference" "U405"
 			(at 52.07 165.1 0)
 			(effects
@@
 			(project "esp-card"
 				(path "/93cf1a11-1660-4ae3-a523-02ca090cff0a/8f237209-f932-45f7-b7bc-f97443ee2306"
-					(reference "U67")
+					(reference "U405")
 					(unit 1)
 				)
@@
 		(dnp no)
 		(fields_autoplaced yes)
-		(property "Reference" "U61"
+		(property "Reference" "U402"
 			(at 52.07 69.85 0)
 			(effects
@@
 			(project "esp-card"
 				(path "/93cf1a11-1660-4ae3-a523-02ca090cff0a/8f237209-f932-45f7-b7bc-f97443ee2306"
-					(reference "U61")
-					(unit 1)
-				)
+					(reference "U402")
+					(unit 1)
+				)
