File: LED_matrix.kicad_sch (KiCad schematic)
At the start: 4 parts, among them U6 NH-B1010RGBT-HF, U7 NH-B1010RGBT-HF, U8 NH-B1010RGBT-HF, U9 NH-B1010RGBT-HF

Commit message: feat: led matrix placed
Parts:
- added U10, U11, U12, U13, U14, U15, U16, U17, U18, U19, U20, U21, U22, U23, U24, U25, U26, U27, U28, U29, U30, U31, U32, U33, U34, U35, U36, U37, U38, U39, U40, U41, U42, U43, U44, U45, U46, U47, U48, U49, U50, U51, U52, U53, U54, U55, U56, U57: NH-B1010RGBT-HF, footprint:LED-ARRAY-SMD_4P-L1.0-W1.0-TR_NH-B1010RGBT, symbol NH-B1010RGBT-HF:NH-B1010RGBT-HF
Connections:
- net CTRL1: now also U6.2 (-), U10.1 (+), U11.1 (+), U12.1 (+), U13.1 (+), U14.3 (-), U18.3 (-), U19.3 (-), U26.3 (-), U27.3 (-), U28.3 (-), U29.3 (-), U42.3 (-), U43.3 (-), U44.3 (-), U45.3 (-)
- net CTRL10: now also U9.2 (-), U43.1 (+), U47.1 (+), U51.1 (+), U55.1 (+)
- net CTRL11: now also U9.3 (-), U44.1 (+), U48.1 (+), U52.1 (+), U56.1 (+)
- net CTRL12: now also U9.4 (-), U45.1 (+), U49.1 (+), U53.1 (+), U57.1 (+)
- net CTRL2: now also U6.3 (-), U10.3 (-), U14.1 (+), U15.1 (+), U16.1 (+), U17.1 (+), U18.4 (-), U19.4 (-), U26.4 (-), U27.4 (-), U28.4 (-), U29.4 (-), U42.4 (-), U43.4 (-), U44.4 (-), U45.4 (-)
- net CTRL3: now also U6.4 (-), U10.4 (-), U14.4 (-), U18.1 (+), U20.1 (+), U21.2 (-), U22.1 (+), U24.1 (+), U30.2 (-), U31.2 (-), U32.2 (-), U33.2 (-), U46.2 (-), U47.2 (-), U48.2 (-), U49.2 (-)
- net CTRL4: now also U7.2 (-), U11.2 (-), U15.2 (-), U19.1 (+), U20.2 (-), U21.1 (+), U23.1 (+), U25.1 (+), U30.3 (-), U31.3 (-), U32.3 (-), U33.3 (-), U46.3 (-), U47.3 (-), U48.3 (-), U49.3 (-)
- net CTRL5: now also U7.3 (-), U11.3 (-), U15.3 (-), U20.3 (-), U21.3 (-), U26.1 (+), U30.1 (+), U31.4 (-), U32.4 (-), U33.4 (-), U34.1 (+), U38.1 (+), U46.4 (-), U47.4 (-), U48.4 (-), U49.4 (-)
- net CTRL6: now also U27.1 (+), U31.1 (+), U35.1 (+), U39.1 (+)
- net CTRL7: now also U8.2 (-), U28.1 (+), U32.1 (+), U36.1 (+), U40.1 (+)
- net CTRL8: now also U8.3 (-), U29.1 (+), U33.1 (+), U37.1 (+), U41.1 (+)
- net CTRL9: now also U8.4 (-), U42.1 (+), U46.1 (+), U50.1 (+), U54.1 (+)
- net at U7.4 (-): now also U11.4 (-), U15.4 (-), U20.4 (-), U21.4 (-), U30.4 (-)
- new net: U10.2 (-), U14.2 (-), U18.2 (-), U19.2 (-), U26.2 (-), U27.2 (-), U28.2 (-), U29.2 (-), U42.2 (-), U43.2 (-), U44.2 (-), U45.2 (-)
Other:
- moved on the sheet: U6

Commit message: feat: led matrix wiring finished
Connections:
- net CTRL0: now also U10.2 (-), U14.2 (-), U18.2 (-), U19.2 (-), U26.2 (-), U27.2 (-), U28.2 (-), U29.2 (-), U42.2 (-), U43.2 (-), U44.2 (-), U45.2 (-)
- net CTRL10: now also U13.2 (-), U17.2 (-), U24.2 (-), U25.2 (-), U38.2 (-), U39.2 (-), U40.2 (-), U41.2 (-), U54.2 (-), U56.3 (-), U57.3 (-)
- net CTRL11: now also U13.3 (-), U17.3 (-), U24.3 (-), U25.3 (-), U38.3 (-), U39.3 (-), U40.3 (-), U41.3 (-), U54.3 (-), U55.3 (-), U57.4 (-)
- net CTRL12: now also U13.4 (-), U17.4 (-), U24.4 (-), U25.4 (-), U38.4 (-), U39.4 (-), U40.4 (-), U41.4 (-), U54.4 (-), U55.4 (-), U56.4 (-)
- net CTRL6: now also U11.4 (-), U15.4 (-), U20.4 (-), U21.4 (-), U30.4 (-), U36.2 (-), U37.2 (-), U50.2 (-), U51.2 (-), U52.2 (-), U53.2 (-), U7.4 (-)
- net CTRL7: now also U12.2 (-), U16.2 (-), U22.2 (-), U23.2 (-), U34.2 (-), U35.2 (-), U37.3 (-), U50.3 (-), U51.3 (-), U52.3 (-), U53.3 (-)
- net CTRL8: now also U12.3 (-), U16.3 (-), U22.3 (-), U23.3 (-), U34.3 (-), U35.3 (-), U36.3 (-), U50.4 (-), U51.4 (-), U52.4 (-), U53.4 (-)
- net CTRL9: now also U12.4 (-), U16.4 (-), U22.4 (-), U23.4 (-), U34.4 (-), U35.4 (-), U36.4 (-), U37.4 (-), U55.2 (-), U56.2 (-), U57.2 (-)

Commit message: led matrix cleanup
Other:
- note added: "Made by @icanc"
- note added: "row 1"
- note added: "row 12"
- note added: "row 3"
- note added: "row 6"
- note added: "row 9"
Changed lines of the file:
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@@
 	(bus
 		(pts
-			(xy 63.5 127) (xy 68.58 127)
+			(xy 63.5 123.19) (xy 68.58 123.19)
 		)
 		(stroke
@@
 	(bus
 		(pts
-			(xy 63.5 92.71) (xy 63.5 127)
+			(xy 63.5 92.71) (xy 63.5 123.19)
 		)
 		(stroke
@@
 	(bus
 		(pts
-			(xy 68.58 127) (xy 68.58 132.08)
+			(xy 68.58 123.19) (xy 68.58 132.08)
 		)
 		(stroke
@@
 		)
 	)
+	(text "row 9"
+		(exclude_from_sim no)
+		(at 92.202 396.494 0)
+		(effects
+			(font
+				(size 1.27 1.27)
+			)
+		)
+	)
+	(text "row 6"
+		(exclude_from_sim no)
+		(at 90.17 294.386 0)
+		(effects
+			(font
+				(size 1.27 1.27)
+			)
+		)
+	)
+	(text "row 12"
+		(exclude_from_sim no)
+		(at 89.154 498.348 0)
+		(effects
+			(font
+				(size 1.27 1.27)
+			)
+		)
+	)
+	(text "row 3"
+		(exclude_from_sim no)
+		(at 94.488 187.452 0)
+		(effects
+			(font
+				(size 1.27 1.27)
+			)
+		)
+	)
+	(text "Made by @icanc"
+		(exclude_from_sim no)
+		(at 388.874 23.368 0)
+		(effects
+			(font
+				(size 1.27 1.27)
+			)
+		)
+	)
+	(text "row 1"
+		(exclude_from_sim no)
+		(at 102.616 110.744 0)
+		(effects
+			(font
+				(size 1.27 1.27)
+			)
+		)
+	)
 	(label "CTRL1"
 		(at 90.17 132.08 0)
@@
 		)
 	)
-	(label "row 1"
-		(at 102.87 114.3 0)
-		(fields_autoplaced yes)
-		(effects
-			(font
-				(size 1.27 1.27)
-			)
-			(justify left bottom)
-		)
-	)
 	(label "CTRL1"
 		(at 255.27 86.36 0)
@@
 		)
 	)
-	(label "row 6"
-		(at 81.28 294.64 0)
-		(fields_autoplaced yes)
-		(effects
-			(font
-				(size 1.27 1.27)
-			)
-			(justify left bottom)
-		)
-	)
 	(label "CTRL11"
 		(at 255.27 45.72 0)
@@
 		)
 	)
-	(label "row 3"
-		(at 83.82 186.69 0)
-		(fields_autoplaced yes)
-		(effects
-			(font
-				(size 1.27 1.27)
-			)
-			(justify left bottom)
-		)
-	)
 	(label "CTRL6"
 		(at 90.17 144.78 0)
@@
 		)
 	)
-	(label "CTRL[0..12]"
-		(at 68.58 127 0)
-		(fields_autoplaced yes)
-		(effects
-			(font
-				(size 1.27 1.27)
-			)
-			(justify left bottom)
-		)
-	)
 	(label "CTRL0"
 		(at 256.54 90.17 0)
@@
 		)
 	)
-	(label "row 9"
-		(at 81.28 397.51 0)
-		(fields_autoplaced yes)
-		(effects
-			(font
-				(size 1.27 1.27)
-			)
-			(justify left bottom)
-		)
-	)
 	(label "CTRL11"
 		(at 90.17 157.48 0)
@@
 		)
 	)
-	(label "made by @icanc"
-		(at 384.81 19.05 0)
-		(fields_autoplaced yes)
-		(effects
-			(font
-				(size 1.27 1.27)
-			)
-			(justify left bottom)
-		)
-	)
 	(label "CTRL10"
 		(at 90.17 154.94 0)
@@
 		)
 	)
+	(hierarchical_label "CTRL[0..12]"
+		(shape tri_state)
+		(at 68.58 123.19 0)
+		(fields_autoplaced yes)
+		(effects
+			(font
+				(size 1.27 1.27)
+			)
+			(justify left)
+		)
+	)

Commit message: fix: led matrix clean up with bus notation
Other:
- moved on the sheet: U10, U11, U12, U13, U14, U15, U16, U17, U18, U19, U20, U21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

Commit message: symbol fixes + placement
Parts:
- renumbered U19 to U10, U26 to U11, U27 to U12, U28 to U13, U29 to U14, U42 to U15, U43 to U16, U44 to U17, U45 to U18, U7 to U19, U11 to U20, U15 to U21, U20 to U22, U21 to U23, U30 to U24, U31 to U25, U32 to U26, U33 to U27, U46 to U28, U47 to U29, U48 to U30, U49 to U31, U8 to U32, U12 to U33, U16 to U34, U22 to U35, U23 to U36, U34 to U37, U35 to U38, U36 to U39, U37 to U40, U50 to U41, U51 to U42, U52 to U43, U53 to U44, U9 to U45, U13 to U46, U17 to U47, U24 to U48, U25 to U49, U38 to U50, U39 to U51, U40 to U52, U41 to U53, U10 to U7, U14 to U8, U18 to U9

Commit message: finished up routing
Parts:
- renumbered U6 to U1, U15 to U10, U16 to U11, U17 to U12, U18 to U13, U19 to U14, U20 to U15, U21 to U16, U22 to U17, U23 to U18, U24 to U19, U7 to U2, U25 to U20, U26 to U21, U27 to U22, U28 to U23, U29 to U24, U30 to U25, U31 to U26, U32 to U27, U33 to U28, U34 to U29, U8 to U3, U35 to U30, U36 to U31, U37 to U32, U38 to U33, U39 to U34, U40 to U35, U41 to U36, U42 to U37, U43 to U38, U44 to U39, U9 to U4, U45 to U40, U46 to U41, U47 to U42, U48 to U43, U49 to U44, U50 to U45, U51 to U46, U52 to U47, U53 to U48, U54 to U49, U10 to U5, U55 to U50, U56 to U51, U57 to U52, U11 to U6, U12 to U7, U13 to U8, U14 to U9
